File: FPVSoundLogger_V2.kicad_sch (KiCad schematic)
At the start: 24 parts, among them J1 USB_C_Receptacle_USB2.0_16P, J2 Conn_01x04, U1 ESP32-S3-MINI-1U, U2 INMP441/IVENSENSE-I2S, U3 XTSD08G, U4 MIC5504-3.3YM5, U5 TPS73633DBV

Commit message: v1.0
Parts:
- removed C2, C3, C4, C5: 10uF/X5R, symbol Device:C
- removed R3, R4, R5: ~, symbol Device:R
- removed R6: 10 kΩ, symbol Device:R
- removed RGBLED: SK6812MINI, LED_SMD:LED_SK6812MINI_PLCC4_3.5x3.5mm_P1.75mm, symbol LED:SK6812MINI
- removed U4: MIC5504-3.3YM5, Package_TO_SOT_SMD:SOT-23-5, symbol Regulator_Linear:MIC5504-3.3YM5
- removed U5: TPS73633DBV, Package_TO_SOT_SMD:SOT-23-5, symbol Regulator_Linear:TPS73633DBV
- added C11: 100nF/16V/X7R, Capacitor_SMD:C_0402_1005Metric_Pad0.74x0.62mm_HandSolder, symbol Device:C
- added C20: 1uF/16V/X7R, Capacitor_SMD:C_0603_1608Metric_Pad1.08x0.95mm_HandSolder, symbol Device:C
- added C21: 10uF/16V/X7R, Capacitor_SMD:C_0603_1608Metric_Pad1.08x0.95mm_HandSolder, symbol Device:C
- added C40, C50, C90, C91: 100nF/10V/X7R, Capacitor_SMD:C_0402_1005Metric_Pad0.74x0.62mm_HandSolder, symbol Device:C
- added D40: 1N4148W, Diode_SMD:D_SOD-123, symbol Diode:1N4148W
- added D6: WS2812B, PCM_JLCPCB:LED_WS2812B_PLCC4_5.0x5.0mm_P3.2mm, symbol PCM_JLCPCB-Extended:LED, WS2812B, 5050
- added D60: Red, PCM_JLCPCB:D_0603, symbol PCM_JLCPCB-Diodes:LED,0603,Red
- added D80: B5819, Diode_SMD:D_SOD-323_HandSoldering, symbol Diode:1N5819
- added H1: MountingHole, MountingHole:MountingHole_3.2mm_M3, symbol Mechanical:MountingHole
- added J3: Conn_01x06, Connector_PinHeader_1.00mm:PinHeader_1x06_P1.00mm_Vertical, symbol Connector_Generic:Conn_01x06
- added R10, R11: 5.1kΩ, Resistor_SMD:R_0603_1608Metric_Pad0.98x0.95mm_HandSolder, symbol Device:R
- added R40: 4.7kΩ, Resistor_SMD:R_0603_1608Metric_Pad0.98x0.95mm_HandSolder, symbol Device:R
- added R41: 0R, Resistor_SMD:R_0603_1608Metric_Pad0.98x0.95mm_HandSolder, symbol Device:R
- added R50: 10kΩ, Resistor_SMD:R_0603_1608Metric_Pad0.98x0.95mm_HandSolder, symbol Device:R
- added R51, R52, R53: ~, Resistor_SMD:R_0603_1608Metric_Pad0.98x0.95mm_HandSolder, symbol Device:R
- added R60: 1kΩ, Resistor_SMD:R_0603_1608Metric_Pad0.98x0.95mm_HandSolder, symbol Device:R
- added R90: 10 kΩ, Resistor_SMD:R_0603_1608Metric_Pad0.98x0.95mm_HandSolder, symbol Device:R
- added U6: AMS1117-3.3, Package_TO_SOT_SMD:SOT-223-3_TabPin2, symbol Regulator_Linear:AMS1117-3.3
- C10: renamed from C1; value 10uF/25V -> 10uF/16V/X7R; footprint (none) -> Capacitor_SMD:C_0805_2012Metric_Pad1.18x1.45mm_HandSolder
- C30: renamed from C6; value 0.1uF/X7R -> 100nF/10V/X7R; footprint (none) -> Capacitor_SMD:C_0402_1005Metric_Pad0.74x0.62mm_HandSolder
- D10: renamed from D1; value 1N5819 -> B5819; footprint Diode_THT:D_DO-41_SOD81_P10.16mm_Horizontal -> Diode_SMD:D_SOD-323_HandSoldering
- D11: renamed from D2; footprint (none) -> Resistor_SMD:R_0603_1608Metric_Pad0.98x0.95mm_HandSolder
- D12: renamed from D3; footprint (none) -> Resistor_SMD:R_0603_1608Metric_Pad0.98x0.95mm_HandSolder
- D13: renamed from D4; footprint (none) -> Resistor_SMD:R_0603_1608Metric_Pad0.98x0.95mm_HandSolder
- J1: footprint (none) -> Connector_USB:USB_C_Receptacle_HRO_TYPE-C-31-M-12
- J2: footprint Connector_JST:JST_EH_B4B-EH-A_1x04_P2.50mm_Vertical -> Connector_JST:JST_SH_SM04B-SRSS-TB_1x04-1MP_P1.00mm_Horizontal
- R30: renamed from R1; value 100 kΩ -> 100kΩ; footprint (none) -> Resistor_SMD:R_0603_1608Metric_Pad0.98x0.95mm_HandSolder
- R54: renamed from R2; footprint (none) -> Resistor_SMD:R_0603_1608Metric_Pad0.98x0.95mm_HandSolder
- U1: footprint PCM_Espressif:ESP32-S3-MINI-1 -> PCM_Espressif:ESP32-S3-MINI-1U
- U2: footprint ProLib_pcs_2025-12-16:MID-SMD_L4.7-W3.8_INMP441ACEZ -> FPVSoundLogger_HW:MIC_INMP441ACEZ-R7
Connections:
- net GND: now also C11.2, C20.2, C21.2, C40.2, C50.2, C90.2, C91.2, D6.3 (VSS), D60.1, J3.3 (Pin_3), R10.1, R11.1, U6.1 (GND)
- net RGB_CTRL: now also D40.1 (K)
- net SDIO_CMD: now also U3.5 (CMD/DI), R52.2; no longer R54.2, U1.28 (SPIIO4/GPIO33/FSPIHD/SUBSPIHD), U1.29 (SPIIO5/GPIO34/FSPICS0/SUBSPICS0), U1.33 (SPIDQS/GPIO37/FSPIQ/SUBSPIQ), U1.34 (GPIO38/FSPIWP/SUBSPIWP)
- net +3V3: now reaches R54.1
- net +3V3: now also C30.1, U1.3 (3V3), U2.7 (VDD), U2.8 (CHIPEN), U3.8 (VDD), C21.1, C50.1, C91.1, J3.1 (Pin_1), R50.1, R51.1, R52.1, R53.1, R60.2, R90.1, U6.2 (VO); no longer U3.1 (SD2)
- net SDIO_DATA_3: now reaches U3.2 (SD3/~{CS})
- net SDIO_DATA_3: now also U1.29 (SPIIO5/GPIO34/FSPICS0/SUBSPICS0), R51.2
- net SDIO_DATA_0: now reaches U3.6 (SD0/DO)
- net SDIO_DATA_0: now also U1.33 (SPIDQS/GPIO37/FSPIQ/SUBSPIQ), R53.2
- net SDIO_DATA_1: now reaches U3.7 (SD1)
- net SDIO_DATA_1: now also R54.2, U1.34 (GPIO38/FSPIWP/SUBSPIWP)
- net VBUS: now reaches D10.2 (A), D11.2 (A2), J1.A4 (VBUS), J1.A9 (VBUS), J1.B4 (VBUS), J1.B9 (VBUS)
- net at J1.A5 (CC1): now also R10.2
- net at J1.B5 (CC2): now also R11.2
- net +5V: now reaches C10.1, D10.1 (K)
- net +5V: now also C11.1, C20.1, C40.1, D6.1 (VDD), D80.1 (K), R40.2, U6.3 (VI)
- net U0TXD: now reaches U1.39 (U0TXD/GPIO43/CLK_OUT1)
- net U0TXD: now also J3.5 (Pin_5)
- net GPIO0/BOOT: now reaches U1.4 (GPIO0/BOOT)
- net U0RXD: now reaches U1.40 (U0RXD/GPIO44/CLK_OUT2)
- net U0RXD: now also J3.6 (Pin_6)
- net EN: now reaches U1.45 (EN)
- net EN: now also C90.1, J3.4 (Pin_4), R90.2
- net VCC_5V: no longer names the net of J2.1 (Pin_1)
- net VCC_5V: now also D80.2 (A)
- new net: D60.2, R60.1
- new net: D40.2 (A), R40.1, R41.1
- new net: D6.4 (DIN), R41.2
- new net GPIO0/BOOT: J3.2 (Pin_2)
- new net SDIO_DATA_2: R50.2, U1.28 (SPIIO4/GPIO33/FSPIHD/SUBSPIHD), U3.1 (SD2)
- no-connect marks 6 -> 25
Other:
- moved on the sheet: C10, C30, D10, D11, D12, D13, J1, J2, R30, R54, U1, U2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
