File: FPVSoundLogger_V2.kicad_pcb (KiCad board)
At the start: 2 copper layers, 38.5 x 38.5 mm, 40 parts, among them J1 USB_C_Receptacle_USB2.0_16P, J2 Conn_01x04, J3 Conn_01x06, U1 ESP32-S3-MINI-1U

Commit message: version sans err drc
Routing:
- net VBUS: track 15.4 -> 22.1 mm
- net I2S_SD: track 52.0 -> 55.7 mm
- net I2S_WS: track 49.7 -> 52.9 mm
- net USB_D-: track 17.3 -> 20.2 mm
- net USB_D+: track 17.7 -> 20.6 mm
- net I2S_SCK: track 49.8 -> 50.9 mm
- net GND: vias 30 -> 29
